Commit message: fix: place lidar above robot collision body

File: ros2_ws/src/substation_description/urdf/inspection_robot.urdf.xacro (robot description, xacro)
@@ -26,5 +26,5 @@
   <joint name="laser_joint" type="fixed">
     <parent link="base_link"/><child link="laser_frame"/>
-    <origin xyz="-0.064 0 0.121" rpy="0 0 0"/>
+    <origin xyz="-0.064 0 0.20" rpy="0 0 0"/>
   </joint>
 </robot>

Commit message: fix: stabilize inspection robot ground support

File: ros2_ws/src/substation_description/urdf/inspection_robot.urdf.xacro (robot description, xacro)
@@ -3,7 +3,7 @@
   <link name="base_footprint"/>
   <link name="base_link">
-    <visual><origin xyz="-0.032 0 0.084"/><geometry><mesh filename="package://turtlebot3_description/meshes/bases/waffle_pi_base.stl" scale="0.001 0.001 0.001"/></geometry></visual>
-    <collision><origin xyz="-0.032 0 0.084"/><geometry><box size="0.28 0.30 0.16"/></geometry></collision>
-    <inertial><origin xyz="0 0 0.08"/><mass value="1.3729096"/><inertia ixx="0.02" ixy="0" ixz="0" iyy="0.02" iyz="0" izz="0.03"/></inertial>
+    <visual><origin xyz="-0.064 0 0"/><geometry><mesh filename="package://turtlebot3_description/meshes/bases/waffle_pi_base.stl" scale="0.001 0.001 0.001"/></geometry></visual>
+    <collision><origin xyz="-0.064 0 0.048"/><geometry><box size="0.265 0.265 0.089"/></geometry></collision>
+    <inertial><origin xyz="-0.064 0 0.048"/><mass value="1.3729096"/><inertia ixx="0.042111447" ixy="0" ixz="0" iyy="0.042111447" iyz="0" izz="0.075254874"/></inertial>
   </link>
   <joint name="base_joint" type="fixed">
@@ -26,5 +26,5 @@
   <joint name="laser_joint" type="fixed">
     <parent link="base_link"/><child link="laser_frame"/>
-    <origin xyz="-0.064 0 0.20" rpy="0 0 0"/>
+    <origin xyz="-0.064 0 0.121" rpy="0 0 0"/>
   </joint>
 </robot>
